File: ESP32-c3-02.kicad_sch (KiCad schematic)
At the start: 23 parts, among them J3 GSD090012SEU, U3 ESP32-C3-WROOM-02-H4, U4 CP2102N-Axx-xQFN20, U5 USBLC6-2SC6, U6 W25Q32JVSSIQ

Commit message: Schematic
Parts:
- added C14: 0.1u, symbol Device:C
- added R22: 50, symbol Device:R
- added TP1: TEST MISO, symbol Connector:TestPoint
- added TP2: TEST MOSI, symbol Connector:TestPoint
- added TP3: TEST SCLK, symbol Connector:TestPoint
- added TP4: TEST CS_SD, symbol Connector:TestPoint
- added TP5: TEST CS, symbol Connector:TestPoint
- renumbered R15 to R16
Connections:
- net +3.3V: now also U6.3 (~{WP}(IO2)), U6.7 (~{HOLD}/~{RESET}(IO3)), U6.8 (VCC), C14.1
- net CS: now also U6.1 (~{CS}), TP5.1
- net CS_SD: now also TP4.1
- net GND: now also U4.12 (GND), U4.21 (GND), U4.3 (GND), U6.4 (GND), C14.2
- net MISO_DO: now also R22.1, TP1.1
- net MOSI_DI: now also U6.5 (DI(IO0)), TP2.1
- net SCLK: now also U6.6 (CLK), TP3.1
- net at U6.2 (DO(IO1)): now also R22.2
- net DTS renamed DTR
Other:
- added sheet Sensor (sensor.kicad_sch)
- added sheet user_interface (user_interface.kicad_sch)
- note added: "Flash memory"
- note added: "SD_Card"
- note added: "TEST"
- title: (none) -> ESP_32
- moved on the sheet: C12, C13, C7, C8, J3, R16, R19, R20, U3, U4, U6

Commit message: schematic1
Parts:
- C10, C11, C12, C14, C8: footprint (none) -> Capacitor_SMD:C_0805_2012Metric
- C13, C7, C9: footprint (none) -> Footprints:T491A
- LED5: value LTST-C170KRKT -> Red; footprint LEDC2012X120N -> Footprints:LEDC2012X120N
- LED6: value LTST-C170GKT -> Green; footprint LEDC2012X120N -> Footprints:LEDC2012X120N
- R11, R12, R13, R14, R15, R16, R19, R20, R22: footprint (none) -> Resistor_SMD:R_0805_2012Metric
- R18: renamed from R16; footprint (none) -> Resistor_SMD:R_0805_2012Metric
- TP1, TP2, TP3, TP4, TP5: footprint (none) -> TestPoint:TestPoint_Pad_D1.0mm
Connections:
- net at R14.1: now also U4.20 (~{TXT}/GPIO.2); no longer U4.19 (~{RXT}/GPIO.3)
- net at R14.2: now also LED6.1 (K); no longer LED5.1 (K)
- net at R15.1: now also U4.19 (~{RXT}/GPIO.3); no longer U4.20 (~{TXT}/GPIO.2)
- net at R15.2: now also LED5.1 (K); no longer LED6.1 (K)
- no-connect marks 5 -> 7
Other:
- moved on the sheet: C12, C13, J3, LED5, LED6, R14, R15, R16, R19

Commit message: intial_PCB
Parts:
- J3: footprint GSD090012SEU:AMPHENOL_GSD090012SEU -> Footprints:AMPHENOL_GSD090012SEU
- U3: footprint ESP32-C3-WROOM-02-H4:MODULE_ESP32-C3-WROOM-02-H4 -> Footprints:MODULE_ESP32-C3-WROOM-02-H4
- U4: footprint Package_DFN_QFN:SiliconLabs_QFN-20-1EP_3x3mm_P0.5mm -> Package_DFN_QFN:SiliconLabs_QFN-20-1EP_3x3mm_P0.5mm_EP1.8x1.8mm
- U6: footprint W25Q32JVSSIQ:SOIC127P790X216-8N -> Footprints:SOIC127P790X216-8N
Connections:
- net CS_SD: now also U3.4 (IO5); no longer U3.18 (IO0)
- net MIC_OUT: now also U3.18 (IO0); no longer U3.4 (IO5)
Changed lines of the file:
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@@
 	)
 	(label "CS_SD"
-		(at 204.47 50.8 180)
+		(at 204.47 63.5 180)
 		(effects
 			(font
@@
 	)
 	(label "MIC_OUT"
-		(at 204.47 63.5 180)
+		(at 204.47 50.8 180)
 		(effects
 			(font
@@
 			)
 		)
-		(property "Footprint" "Package_DFN_QFN:SiliconLabs_QFN-20-1EP_3x3mm_P0.5mm"
+		(property "Footprint" "Package_DFN_QFN:SiliconLabs_QFN-20-1EP_3x3mm_P0.5mm_EP1.8x1.8mm"
 			(at 113.03 107.95 0)
 			(effects
@@
 			)
 		)
-		(property "Footprint" "W25Q32JVSSIQ:SOIC127P790X216-8N"
+		(property "Footprint" "Footprints:SOIC127P790X216-8N"
 			(at 76.2 157.48 0)
 			(effects
@@
 			)
 		)
-		(property "Footprint" "GSD090012SEU:AMPHENOL_GSD090012SEU"
+		(property "Footprint" "Footprints:AMPHENOL_GSD090012SEU"
 			(at 201.93 114.3 0)
 			(effects
@@
 			)
 		)
-		(property "Footprint" "ESP32-C3-WROOM-02-H4:MODULE_ESP32-C3-WROOM-02-H4"
+		(property "Footprint" "Footprints:MODULE_ESP32-C3-WROOM-02-H4"
 			(at 222.25 60.96 0)
 			(effects
