File: esp_32.kicad_pcb (KiCad board)
At the start: 4 copper layers, 17 parts, among them J1 USB_B_Micro, U1 ESP32-S3-MINI-1, U2 D3V3XA4B10LP, U3 TLV75801PDRV

Commit message: intial_PCB
Parts:
- removed Boot1, Reset1: SW_MEC_5E, Button_Switch_SMD:SW_DIP_SPSTx02_Slide_6.7x6.64mm_W6.73mm_P2.54mm_LowProfile_JPin
- removed D2: LED, LED_SMD:LED_0603_1608Metric
- added C10: 0.1u, Capacitor_SMD:C_0805_2012Metric, F.Cu at (151.7, 121.2)
- added C11: 1u, Capacitor_SMD:C_0805_2012Metric, F.Cu at (143.2, 110.8)
- added C12: 0.1u, Capacitor_SMD:C_0805_2012Metric, F.Cu at (186.2, 108.8)
- added C13: 10u, Footprints:T491A, F.Cu at (181.2, 108.1)
- added C14: 0.1u, Capacitor_SMD:C_0805_2012Metric, F.Cu at (156.8, 108.5)
- added C15: 0.1u, Capacitor_SMD:C_0805_2012Metric, F.Cu at (152.3, 88.5)
- added C16: 0.1U, Capacitor_SMD:C_0805_2012Metric, F.Cu at (126.2, 87.7)
- added C17: 10n, Capacitor_SMD:C_0805_2012Metric, F.Cu at (137.7, 94.0)
- added C18: 0.1u, Capacitor_SMD:C_0805_2012Metric, F.Cu at (126.8, 90.5)
- added C19: 10u, Capacitor_SMD:C_0805_2012Metric, F.Cu at (120.5, 87.5)
- added C20: 0.1U, Capacitor_SMD:C_0805_2012Metric, F.Cu at (129.6, 101.0)
- added C21: 0.1u, Capacitor_SMD:C_0805_2012Metric, F.Cu at (158.6, 130.6)
- added C22: 1u, Capacitor_SMD:C_0805_2012Metric, F.Cu at (165.0, 130.6)
- added C23: 0.1u, Capacitor_SMD:C_0805_2012Metric, F.Cu at (155.4, 95.5)
- added C24: 10n, Capacitor_SMD:C_0805_2012Metric, F.Cu at (153.7, 99.0)
- added C25: 10n, Capacitor_SMD:C_0805_2012Metric, F.Cu at (146.7, 95.8)
- added C5: 10u, Footprints:T491A, F.Cu at (116.1, 116.6)
- added C8: 0.1u, Capacitor_SMD:C_0805_2012Metric, F.Cu at (198.2, 94.0)
- added C9: 4.7u, Footprints:T491A, F.Cu at (149.8, 115.0)
- added F1: 0ZCH0110AF2E, Footprints:FUSC3226X100N, F.Cu at (132.8, 120.4)
- added FB1: FBMJ2125HM330-T, Footprints:BEADC2012X105N, F.Cu at (119.8, 127.6)
- added J3: GSD090012SEU, Footprints:AMPHENOL_GSD090012SEU, F.Cu at (184.2, 124.3)
- added J4: B4B-XH-AM, Footprints:JST_B4B-XH-AM__LF__SN_, F.Cu at (108.2, 90.8)
- added J5: B2B-PH-SM4-TB, Connector_JST:JST_PH_B2B-PH-K_1x02_P2.00mm_Vertical, F.Cu at (110.3, 132.4)
- added J6: Conn_01x05, Connector_PinHeader_2.54mm:PinHeader_1x05_P2.54mm_Vertical, F.Cu at (108.0, 102.1)
- added LED1: Red, Footprints:LEDC2012X120N, F.Cu at (108.7, 122.3)
- added LED2: Green, Footprints:LEDC2012X120N, F.Cu at (111.9, 122.3)
- added LED3: Blue, Footprints:LEDC2012X120N, F.Cu at (114.9, 122.2)
- added LED4: RED D4, Footprints:LEDC2012X120N, F.Cu at (114.2, 106.3)
- added LED5: Red, Footprints:LEDC2012X120N, F.Cu at (130.9, 108.5)
- added LED6: Green, Footprints:LEDC2012X120N, F.Cu at (135.2, 108.5)
- added MK1: CMC-5042PF-AC, Footprints:CUI_CMC-5042PF-AC, F.Cu at (138.2, 89.2)
- added Q1: TEMT6000X01, Footprints:TRANS_TEMT6000X01, F.Cu at (151.2, 95.3)
- added Q2: BC817, Package_TO_SOT_SMD:SOT-23, F.Cu at (164.7, 121.1)
- added Q3: BC817, Package_TO_SOT_SMD:SOT-23, F.Cu at (158.9, 121.1)
- added R1: 10K, Resistor_SMD:R_0805_2012Metric, F.Cu at (118.4, 122.7)
- added R10: 470, Resistor_SMD:R_0805_2012Metric, F.Cu at (114.6, 102.6)
- added R11: 1K, Resistor_SMD:R_0805_2012Metric, F.Cu at (139.4, 109.2)
- added R12: 22K1, Resistor_SMD:R_0805_2012Metric, F.Cu at (147.8, 109.0)
- added R13: 47K5, Resistor_SMD:R_0805_2012Metric, F.Cu at (143.2, 107.0)
- added R14: 470, Resistor_SMD:R_0805_2012Metric, F.Cu at (134.9, 112.7)
- added R15: 470, Resistor_SMD:R_0805_2012Metric, F.Cu at (130.9, 113.0)
- added R16: 50, Resistor_SMD:R_0805_2012Metric, F.Cu at (176.9, 108.2)
- added R17: 35WR100KLFTR, Footprints:TRIM_35WR100KLFTR, F.Cu at (131.3, 93.8)
- added R18: 50, Resistor_SMD:R_0805_2012Metric, F.Cu at (175.3, 99.0)
- added R19: 10K, Resistor_SMD:R_0805_2012Metric, F.Cu at (191.1, 107.4)
- added R2: 10k, Resistor_SMD:R_0805_2012Metric, F.Cu at (120.9, 122.7)
- added R20: 50, Resistor_SMD:R_0805_2012Metric, F.Cu at (175.2, 96.8)
- added R21: 10K, Resistor_SMD:R_0805_2012Metric, F.Cu at (150.4, 99.1)
- added R22: 50, Resistor_SMD:R_0805_2012Metric, F.Cu at (163.0, 111.5)
- added R24: 4K7, Resistor_SMD:R_0805_2012Metric, F.Cu at (156.2, 85.5)
- added R25: 4K7, Resistor_SMD:R_0805_2012Metric, F.Cu at (158.2, 85.5)
- added R26: 2K, Resistor_SMD:R_0805_2012Metric, F.Cu at (121.1, 96.1)
- added R27: 1m, Resistor_SMD:R_0805_2012Metric, F.Cu at (126.5, 93.8)
- added R28: 2K, Resistor_SMD:R_0805_2012Metric, F.Cu at (131.0, 87.0)
- added R29: 1m, Resistor_SMD:R_0805_2012Metric, F.Cu at (131.6, 97.8)
- added R30: 1k, Resistor_SMD:R_0805_2012Metric, F.Cu at (121.8, 91.5)
- added R31: 22K, Resistor_SMD:R_0805_2012Metric, F.Cu at (126.8, 97.5)
- added R32: 10K, Resistor_SMD:R_0805_2012Metric, F.Cu at (154.0, 133.1)
- added R33: 10K, Resistor_SMD:R_0805_2012Metric, F.Cu at (158.9, 126.8)
- added R34: 10K, Resistor_SMD:R_0805_2012Metric, F.Cu at (164.4, 126.6)
- added R4: 5k1, Resistor_SMD:R_0805_2012Metric, F.Cu at (145.6, 115.3)
- added R5: 2k, Resistor_SMD:R_0805_2012Metric, F.Cu at (123.4, 122.7)
- added R9: 470, Resistor_SMD:R_0805_2012Metric, F.Cu at (114.7, 126.8)
- added S1: BOOT, Footprints:SW_USLPT2819DT2TR, F.Cu at (158.3, 134.4)
- added S2: RESET, Footprints:SW_USLPT2819DT2TR, F.Cu at (164.8, 134.6)
- added TP1: TEST MISO, TestPoint:TestPoint_Pad_D1.0mm, F.Cu at (246.0, 114.3)
- added TP2: TEST MOSI, TestPoint:TestPoint_Pad_D1.0mm, F.Cu at (241.8, 119.0)
- added TP3: TEST SCLK, TestPoint:TestPoint_Pad_D1.0mm, F.Cu at (241.2, 128.8)
- added TP4: TEST CS_SD, TestPoint:TestPoint_Pad_D1.0mm, F.Cu at (234.7, 110.5)
- added TP5: TEST CS, TestPoint:TestPoint_Pad_D1.0mm, F.Cu at (230.2, 94.6)
- added U4: CP2102N-Axx-xQFN20, Package_DFN_QFN:SiliconLabs_QFN-20-1EP_3x3mm_P0.5mm_EP1.8x1.8mm, F.Cu at (139.9, 114.8)
- added U5: USBLC6-2SC6, Package_TO_SOT_SMD:SOT-23-6, F.Cu at (139.1, 120.5)
- added U6: W25Q32JVSSIQ, Footprints:SOIC127P790X216-8N, F.Cu at (162.8, 107.5)
- added U7: MAX4466EXK, Footprints:SOT65P210X110-5N, F.Cu at (131.0, 90.1)
- added VR1: LM1117MPX-3.3, Footprints:VREG_LM1117MPX-3.3, F.Cu at (119.6, 109.6)
- C1, C4: value 0.1uf -> 0.1u; footprint Capacitor_SMD:C_0603_1608Metric -> Capacitor_SMD:C_0805_2012Metric
- C2: value 10uf -> 0.1u; footprint Capacitor_SMD:C_0603_1608Metric -> Capacitor_SMD:C_0805_2012Metric
- C3: value 0.1uf -> 10u; footprint Capacitor_SMD:C_0603_1608Metric -> Footprints:T491A
- C6: value 10uf -> 1u; footprint Capacitor_SMD:C_0603_1608Metric -> Capacitor_SMD:C_0805_2012Metric
- C7: value 10uf -> 10u; footprint Capacitor_SMD:C_0603_1608Metric -> Footprints:T491A
- J1: value USB_B_Micro -> SS-52400-002; footprint Connector_USB:USB_Micro-B_Molex-105017-0001 -> Footprints:BELFUSE_SS-52400-002
- R3: value 10k -> 5k1; footprint Resistor_SMD:R_0603_1608Metric -> Resistor_SMD:R_0805_2012Metric
- R6: value 1M -> 20k; footprint Resistor_SMD:R_0603_1608Metric -> Resistor_SMD:R_0805_2012Metric
- R7: value 200k -> 470; footprint Resistor_SMD:R_0603_1608Metric -> Resistor_SMD:R_0805_2012Metric
- R8: value 5.1k -> 470; footprint Resistor_SMD:R_0603_1608Metric -> Resistor_SMD:R_0805_2012Metric
- U1: value ESP32-S3-MINI-1 -> MCP73871; footprint RF_Module:ESP32-S2-MINI-1 -> Package_DFN_QFN:QFN-20-1EP_4x4mm_P0.5mm_EP2.5x2.5mm
- U2: value D3V3XA4B10LP -> BME280; footprint Package_DFN_QFN:Diodes_UDFN-10_1.0x2.5mm_P0.5mm -> Footprints:PSON65P250X250X100-8N
- U3: value TLV75801PDRV -> ESP32-C3-WROOM-02-H4; footprint Package_SON:WSON-6-1EP_2x2mm_P0.65mm_EP1x1.6mm -> Footprints:MODULE_ESP32-C3-WROOM-02-H4
- moved R7 77.8 mm to (108.7, 126.8), turned to 90 degrees
- moved R8 74.0 mm to (111.7, 126.8), turned to 90 degrees
- moved C4 63.9 mm to (113.8, 111.9), turned to -90 degrees
- moved R6 61.6 mm to (125.9, 122.6), turned to 90 degrees
- moved U1 60.9 mm to (120.0, 131.8), turned to -90 degrees
- moved C6 60.1 mm to (123.4, 127.1), turned to -90 degrees
- moved C3 58.1 mm to (122.8, 116.6)
- moved C2 55.3 mm to (124.8, 111.9), turned to -90 degrees
- moved C1 45.8 mm to (144.7, 120.7), turned to 90 degrees
- moved R3 44.3 mm to (148.1, 120.6), turned to 90 degrees
- moved J1 41.9 mm to (138.6, 131.6)
- moved U3 33.9 mm to (187.0, 93.6)
- moved U2 25.0 mm to (152.2, 85.3), turned to 180 degrees
- moved C7 7.27 mm to (175.2, 92.8), turned to -90 degrees
Connections:
- C1 pad 1: /3V3 -> /VBUS
- C2 pad 1: /3V3 -> +5V
- C3 pad 1: /ESP32_EN -> +5V
- C4 pad 1: /GPIOO -> +3.3V
- C6 pad 1: /5VUSB -> GND
- C6 pad 2: GND -> /+5V_USB
- C7 pad 1: /3V3 -> +3.3V
- R3 pad 1: /3V3 -> Net-(J1-CC2)
- R3 pad 2: /ESP32_EN -> GND
- R6 pad 1: /3V3 -> Net-(U1-PROG3)
- R6 pad 2: Net-(U3-FB) -> GND
- R7 pad 1: Net-(U3-FB) -> /Charging
- R7 pad 2: GND -> Net-(LED1-K)
- R8 pad 1: /3V3 -> /Charged
- U1 pad 1: GND -> Net-(FB1-Pad2)
- U1 pad 10: unconnected-(U1-IO6-Pad10) -> GND
- U1 pad 11: unconnected-(U1-IO7-Pad11) -> GND
- U1 pad 12: unconnected-(U1-IO8-Pad12) -> Net-(U1-PROG3)
- U1 pad 13: unconnected-(U1-IO9-Pad13) -> Net-(U1-PROG1)
- U1 pad 14: unconnected-(U1-IO10-Pad14) -> /VBAT
- U1 pad 15: unconnected-(U1-IO11-Pad15) -> /VBAT
- U1 pad 16: unconnected-(U1-IO12-Pad16) -> /VBAT
- U1 pad 17: unconnected-(U1-IO13-Pad17) -> /+5V_USB
- U1 pad 18: unconnected-(U1-IO14-Pad18) -> /+5V_USB
- U1 pad 19: unconnected-(U1-IO15-Pad19) -> /+5V_USB
- U1 pad 2: GND -> /+5V_USB
- U1 pad 20: unconnected-(U1-IO16-Pad20) -> Net-(FB1-Pad2)
- U1 pad 21: unconnected-(U1-IO17-Pad21) -> GND
- U1 pad 3: /3V3 -> GND
- U1 pad 4: /GPIOO -> /+5V_USB
- U1 pad 5: unconnected-(U1-IO1-Pad5) -> Net-(U1-THERM)
- U1 pad 6: unconnected-(U1-IO2-Pad6) -> /Charging_power_good
- U1 pad 7: unconnected-(U1-IO3-Pad7) -> /Charging
- U1 pad 8: unconnected-(U1-IO4-Pad8) -> /Charged
- U1 pad 9: unconnected-(U1-IO5-Pad9) -> Net-(U1-~{TE})
- U2 pad 1: /USB_N -> GND
- U2 pad 2: /USB_P -> +3.3V
- U2 pad 3: GND -> /ESP32-c3-02/SDA
- U2 pad 4: /5VUSB -> /ESP32-c3-02/SCL
- U2 pad 5: unconnected-(U2-Pad5) -> GND
- U2 pad 6: unconnected-(U2-NC-Pad6) -> +3.3V
- U2 pad 7: /5VUSB -> GND
- U2 pad 8: GND -> +3.3V
- U3 pad 1: /3V3 -> +3.3V
- U3 pad 2: Net-(U3-FB) -> /ESP32-c3-02/EN
- U3 pad 3: GND -> /ESP32-c3-02/SDA
- U3 pad 4: /5VUSB -> /ESP32-c3-02/CS_SD
- U3 pad 5: unconnected-(U3-DNC-Pad5) -> Net-(U3-IO6)
- U3 pad 6: /5VUSB -> Net-(U3-IO7)
- U3 pad 7: GND -> /ESP32-c3-02/GPIO8
Other:
- board outline added: 96 x 54 mm
- board text removed: "ESP 32S"
- board text removed: "Kowshik.pvt"
- board text removed: "Made in India"

Commit message: PCB1
Parts:
- added REF**: MountingHole_2.5mm, MountingHole:MountingHole_2.5mm, F.Cu at (119.8, 98.5)
- added REF**: MountingHole_2.5mm, MountingHole:MountingHole_2.5mm, F.Cu at (163.2, 96.2)
- added REF**: MountingHole_2.5mm, MountingHole:MountingHole_2.5mm, F.Cu at (141.8, 101.5)
- moved TP1 80.4 mm to (165.7, 113.7)
- moved TP3 73.7 mm to (171.9, 103.7)
- moved TP2 57.9 mm to (185.7, 105.2)
- moved TP4 46.1 mm to (188.9, 105.2)
- moved TP5 33.8 mm to (198.2, 105.5)
- moved LED1 6.23 mm to (114.9, 122.2)
- moved R7 6.23 mm to (114.9, 127.0)
- moved J5 5.65 mm to (115.8, 133.8), turned to 180 degrees
- moved J4 4.72 mm to (113.0, 90.8)
- moved U1 4.03 mm to (123.9, 132.9), turned to 180 degrees
- moved R15 4.01 mm to (134.9, 113.2)
- moved J6 3.82 mm to (111.8, 102.9)
- moved C17 3.79 mm to (141.1, 95.8)
- moved C18 3.79 mm to (130.2, 92.3)
- moved R26 3.79 mm to (124.4, 97.9)
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Routing:
- net GND: track 0.00 -> 102.9 mm, vias 0 -> 44
- net /ESP32-c3-02/SDA: track 0.00 -> 97.9 mm, vias 0 -> 2
- net /ESP32-c3-02/SCL: track 0.00 -> 97.3 mm, vias 0 -> 2
- net /ESP32-c3-02/GPIO19: track 0.00 -> 90.3 mm, vias 0 -> 1
- net +3.3V: track 0.00 -> 90.3 mm, vias 0 -> 28
- net /ESP32-c3-02/GPIO18: track 0.00 -> 87.8 mm, vias 0 -> 1
- net /ESP32-c3-02/BOOT: track 0.00 -> 86.6 mm, vias 0 -> 2
- net /ESP32-c3-02/MIC_OUT: track 0.00 -> 86.0 mm
- net /ESP32-c3-02/MISO_DO: track 0.00 -> 72.1 mm
- net /ESP32-c3-02/GPIO8: track 0.00 -> 68.6 mm, vias 0 -> 1
- net /ESP32-c3-02/CS: track 0.00 -> 59.8 mm
- net /ESP32-c3-02/MOSI_DI: track 0.00 -> 58.2 mm
- net /ESP32-c3-02/DTR: track 0.00 -> 37.1 mm, vias 0 -> 2
- net /+5V_USB: track 0.00 -> 36.5 mm, vias 0 -> 6
- net /ESP32-c3-02/RTS: track 0.00 -> 36.0 mm, vias 0 -> 2
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- added copper zone on F.Cu, net +3.3V
- added copper zone on In1.Cu, net +3.3V
- added copper zone on F.Cu, net +5V
- added copper zone on F.Cu, net /+5V_USB
- added copper zone on In1.Cu, net /+5V_USB
- added copper zone on F.Cu, net /VBAT
- added copper zone on F.Cu, net /VBUS
- added copper zone on In1.Cu, net /VBUS
- added copper zone on F.Cu, net GND
- added copper zone on In2.Cu, net GND
Other:
- board outline removed

Commit message: finished_PCB
Parts:
- moved REF** 20.5 mm to (161.7, 96.7)
- moved REF** 17.9 mm to (158.4, 113.5)
- moved TP2 12.7 mm to (173.2, 107.5)
- moved MK1 0.60 mm to (141.9, 90.5)
- moved J5 0.32 mm to (115.7, 133.4)
Routing:
- net /ESP32-c3-02/TX_RX: track 0.00 -> 81.7 mm, vias 0 -> 2
- net /ESP32-c3-02/EN: track 30.3 -> 107.3 mm, vias 0 -> 2
- net /ESP32-c3-02/RX_TX: track 0.00 -> 68.7 mm, vias 0 -> 2
- net GND: track 102.9 -> 168.6 mm, vias 44 -> 40
- net /ESP32-c3-02/PHOTO_C: track 13.0 -> 64.7 mm, vias 0 -> 2
- net Net-(U1-PROG3): track 0.00 -> 19.8 mm, vias 0 -> 2
- net Net-(U1-PROG1): track 0.00 -> 18.0 mm, vias 0 -> 2
- net Net-(U1-~{TE}): track 0.00 -> 8.64 mm, vias 0 -> 2
- net /ESP32-c3-02/BOOT: track 86.6 -> 91.2 mm
- net +3.3V: track 90.3 -> 94.8 mm
- net Net-(FB1-Pad2): track 9.41 -> 13.0 mm
- net /ESP32-c3-02/MOSI_DI: track 58.2 -> 55.1 mm
- net /ESP32-c3-02/RTS: track 36.0 -> 38.5 mm
- net /+5V_USB: track 36.5 -> 38.2 mm
- net /VBAT: track 8.67 -> 7.09 mm
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Other:
- board outline added: 93.5 x 58 mm
- board text added: "Battery_charger"
- board text added: "Envinormental_sensor"
- board text added: "KOWSHIK_PVT"
- board text added: "LGO"
- board text added: "OLED display"
- board text added: "SD_Card"
- board text added: "SD_card"
- board text added: "USB"
- board text added: "esp32"
- board text added: "flash_ memory"
- board text added: "micro_phone"
- board text added: "photo_sensor"
- board text added: "rest_boot"
