File: sensor.kicad_sch (KiCad schematic)
At the start: 23 parts, among them Q1 TEMT6000X01, U2 BME280, U7 MAX4466EXK

Commit message: schematic1
Parts:
- C15, C16, C18, C20, C23: footprint (none) -> Capacitor_SMD:C_0805_2012Metric
- C17: renamed from C19; footprint (none) -> Capacitor_SMD:C_0805_2012Metric
- C19: renamed from C17; footprint (none) -> Capacitor_SMD:C_0805_2012Metric
- R17: renamed from R23; footprint Footprints:TRIM_35WR100KLFTR -> Resistor_SMD:R_0805_2012Metric
- R24, R25, R26, R28, R30, R31: footprint (none) -> Resistor_SMD:R_0805_2012Metric
- R27: renamed from R18; footprint (none) -> Resistor_SMD:R_0805_2012Metric
- R29: renamed from R17; footprint (none) -> Resistor_SMD:R_0805_2012Metric
Connections:
- net MIC_OUT: now also C20.2, R17.1, R17.2
Other:
- moved on the sheet: C18
Changed lines of the file:
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@@
 	)
 	(junction
+		(at 240.03 132.08)
+		(diameter 0)
+		(color 0 0 0 0)
+	)
+	(junction
 		(at 182.88 132.08)
 		(diameter 0)
@@
 	)
 	(junction
-		(at 237.49 147.32)
-		(diameter 0)
-		(color 0 0 0 0)
-	)
-	(junction
 		(at 173.99 132.08)
 		(diameter 0)
@@
 	(wire
 		(pts
-			(xy 252.73 134.62) (xy 252.73 142.24)
+			(xy 254 134.62) (xy 254 142.24)
 		)
 		(stroke
@@
 	(wire
 		(pts
-			(xy 252.73 142.24) (xy 247.65 142.24)
+			(xy 254 142.24) (xy 247.65 142.24)
 		)
 		(stroke
@@
 	(wire
 		(pts
-			(xy 237.49 132.08) (xy 237.49 147.32)
+			(xy 68.58 48.26) (xy 68.58 52.07)
 		)
 		(stroke
@@
 	(wire
 		(pts
-			(xy 68.58 48.26) (xy 68.58 52.07)
+			(xy 182.88 104.14) (xy 182.88 121.92)
 		)
 		(stroke
@@
 	(wire
 		(pts
-			(xy 182.88 104.14) (xy 182.88 121.92)
+			(xy 173.99 116.84) (xy 173.99 118.11)
 		)
 		(stroke
@@
 	(wire
 		(pts
-			(xy 173.99 116.84) (xy 173.99 118.11)
+			(xy 203.2 160.02) (xy 213.36 160.02)
 		)
 		(stroke
@@
 	(wire
 		(pts
-			(xy 203.2 160.02) (xy 213.36 160.02)
+			(xy 100.33 77.47) (xy 106.68 77.47)
 		)
 		(stroke
@@
 	(wire
 		(pts
-			(xy 100.33 77.47) (xy 106.68 77.47)
+			(xy 240.03 132.08) (xy 240.03 152.4)
 		)
 		(stroke
@@
 	(wire
 		(pts
+			(xy 241.3 132.08) (xy 240.03 132.08)
+		)
+		(stroke
+			(width 0)
+			(type default)
+		)
+	)
+	(wire
+		(pts
 			(xy 170.18 116.84) (xy 173.99 116.84)
 		)
@@
 	(wire
 		(pts
-			(xy 252.73 127) (xy 247.65 127)
+			(xy 254 127) (xy 247.65 127)
 		)
 		(stroke
@@
 	(wire
 		(pts
+			(xy 240.03 132.08) (xy 238.76 132.08)
+		)
+		(stroke
+			(width 0)
+			(type default)
+		)
+	)
+	(wire
+		(pts
 			(xy 41.91 69.85) (xy 48.26 69.85)
 		)
@@
 	(wire
 		(pts
+			(xy 237.49 152.4) (xy 240.03 152.4)
+		)
+		(stroke
+			(width 0)
+			(type default)
+		)
+	)
+	(wire
+		(pts
 			(xy 157.48 53.34) (xy 162.56 53.34)
 		)
@@
 	(hierarchical_label "MIC_OUT"
 		(shape output)
-		(at 238.76 132.08 0)
+		(at 241.3 132.08 0)
 		(effects
 			(font
@@
 			)
 		)
-		(property "Footprint" ""
+		(property "Footprint" "Capacitor_SMD:C_0805_2012Metric"
 			(at 206.7052 64.77 0)
 			(effects
@@
 			)
 		)
-		(property "Footprint" ""
+		(property "Footprint" "Capacitor_SMD:C_0805_2012Metric"
 			(at 170.18 115.8748 0)
 			(effects
@@
 			)
 		)
-		(property "Footprint" ""
+		(property "Footprint" "Resistor_SMD:R_0805_2012Metric"
 			(at 56.642 59.69 90)
 			(effects
@@
 			)
 		)
-		(property "Footprint" ""
+		(property "Footprint" "Resistor_SMD:R_0805_2012Metric"
 			(at 210.82 154.178 90)
 			(effects
@@
 			)
 		)
-		(property "Footprint" ""
+		(property "Footprint" "Capacitor_SMD:C_0805_2012Metric"
 			(at 107.6452 69.85 0)
 			(effects
@@
 			)
 		)
-		(property "Footprint" ""
+		(property "Footprint" "Resistor_SMD:R_0805_2012Metric"
 			(at 175.768 121.92 90)
 			(effects
@@
 		(on_board yes)
 		(dnp no)
-		(property "Reference" "R23"
+		(property "Reference" "R17"
 			(at 231.648 149.606 0)
 			(effects
@@
 			)
 		)
-		(property "Footprint" "Footprints:TRIM_35WR100KLFTR"
+		(property "Footprint" "Resistor_SMD:R_0805_2012Metric"
 			(at 226.06 152.4 0)
 			(effects
@@
 			(project "esp_32"
 				(path "/db43b58c-fd32-4bba-b73e-41c96465b130/67fd96cd-9b72-43ab-a2ef-5ad5e85521dd/f9d4c426-5fcc-495c-aef9-222a3e6f6529"
-					(reference "R23")
+					(reference "R17")
 					(unit 1)
 				)
@@
 			)
 		)
-		(property "Footprint" ""
+		(property "Footprint" "Resistor_SMD:R_0805_2012Metric"
 			(at 46.482 59.69 90)
 			(effects
@@
 		(dnp no)
 		(fields_autoplaced yes)
-		(property "Reference" "R17"
+		(property "Reference" "R29"
 			(at 185.42 137.1599 0)
 			(effects
@@
 			)
 		)
-		(property "Footprint" ""
+		(property "Footprint" "Resistor_SMD:R_0805_2012Metric"
 			(at 184.658 138.43 90)
 			(effects
@@
 			(project "esp_32"
 				(path "/db43b58c-fd32-4bba-b73e-41c96465b130/67fd96cd-9b72-43ab-a2ef-5ad5e85521dd/f9d4c426-5fcc-495c-aef9-222a3e6f6529"
-					(reference "R17")
+					(reference "R29")
 					(unit 1)
 				)
@@
 			)
 		)
-		(property "Footprint" ""
+		(property "Footprint" "Resistor_SMD:R_0805_2012Metric"
 			(at 175.768 110.49 90)
 			(effects
@@
 		(dnp no)
 		(fields_autoplaced yes)
-		(property "Reference" "C17"
+		(property "Reference" "C19"
 			(at 196.85 144.7799 0)
 			(effects
@@
 			)
 		)
-		(property "Footprint" ""
+		(property "Footprint" "Capacitor_SMD:C_0805_2012Metric"
 			(at 194.0052 149.86 0)
 			(effects
@@
 			(project ""
 				(path "/db43b58c-fd32-4bba-b73e-41c96465b130/67fd96cd-9b72-43ab-a2ef-5ad5e85521dd/f9d4c426-5fcc-495c-aef9-222a3e6f6529"
-					(reference "C17")
+					(reference "C19")
 					(unit 1)
 				)
@@
 		(dnp no)
 		(fields_autoplaced yes)
-		(property "Reference" "R18"
+		(property "Reference" "R27"
 			(at 185.42 124.4599 0)
 			(effects
@@
 			)
 		)
-		(property "Footprint" ""
+		(property "Footprint" "Resistor_SMD:R_0805_2012Metric"
 			(at 184.658 125.73 90)
 			(effects
@@
 			(project "esp_32"
 				(path "/db43b58c-fd32-4bba-b73e-41c96465b130/67fd96cd-9b72-43ab-a2ef-5ad5e85521dd/f9d4c426-5fcc-495c-aef9-222a3e6f6529"
-					(reference "R18")
+					(reference "R27")
 					(unit 1)
 				)
@@
 			)
 		)
-		(property "Footprint" ""
+		(property "Footprint" "Capacitor_SMD:C_0805_2012Metric"
 			(at 220.98 159.0548 0)
 			(effects
@@
 		(on_board yes)
 		(dnp no)
-		(property "Reference" "C19"
+		(property "Reference" "C17"
 			(at 170.18 134.366 90)
 			(effects
@@
 			)
 		)
-		(property "Footprint" ""
+		(property "Footprint" "Capacitor_SMD:C_0805_2012Metric"
 			(at 181.61 131.1148 0)
 			(effects
@@
 			(project "esp_32"
 				(path "/db43b58c-fd32-4bba-b73e-41c96465b130/67fd96cd-9b72-43ab-a2ef-5ad5e85521dd/f9d4c426-5fcc-495c-aef9-222a3e6f6529"
-					(reference "C19")
+					(reference "C17")
 					(unit 1)
 				)
@@
 	(symbol
 		(lib_id "Device:C")
-		(at 252.73 130.81 0)
+		(at 254 130.81 0)
 		(unit 1)
 		(exclude_from_sim no)
@@
 		(fields_autoplaced yes)
 		(property "Reference" "C18"
-			(at 256.54 129.5399 0)
+			(at 257.81 129.5399 0)
 			(effects
 				(font
@@
 		)
 		(property "Value" "0.1u"
-			(at 256.54 132.0799 0)
+			(at 257.81 132.0799 0)
 			(effects
 				(font
@@
 			)
 		)
-		(property "Footprint" ""
-			(at 253.6952 134.62 0)
+		(property "Footprint" "Capacitor_SMD:C_0805_2012Metric"
+			(at 254.9652 134.62 0)
 			(effects
 				(font
@@
 		)
 		(property "Datasheet" "~"
-			(at 252.73 130.81 0)
+			(at 254 130.81 0)
 			(effects
 				(font
@@
 		)
 		(property "Description" "Unpolarized capacitor"
-			(at 252.73 130.81 0)
+			(at 254 130.81 0)
 			(effects
 				(font
@@
 			)
 		)
-		(property "Footprint" ""
+		(property "Footprint" "Resistor_SMD:R_0805_2012Metric"
 			(at 194.818 138.43 90)
 			(effects

Commit message: intial_PCB
Parts:
- C17: value 1u -> 10n
- C19: value 1u -> 10u
- MK1: footprint CMC-5042PF-AC:CUI_CMC-5042PF-AC -> Footprints:CUI_CMC-5042PF-AC
- Q1: footprint TEMT6000X01:TRANS_TEMT6000X01 -> Footprints:TRANS_TEMT6000X01; Check_prices https://www.snapeda.com/parts/TEMT6000X01/Vishay+Semiconduc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 -> https://www.snapeda.com/parts/TEMT6000X01/Vishay/view-part/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; SnapEDA_Link https://www.snapeda.com/parts/TEMT6000X01/Vishay+Semiconduc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 -> https://www.snapeda.com/parts/TEMT6000X01/Vishay/view-part/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
- R17: footprint Resistor_SMD:R_0805_2012Metric -> Footprints:TRIM_35WR100KLFTR
- R27, R29: value 10k -> 1m
- R30: value 10k -> 1k
- U2: footprint BME280:PSON65P250X250X100-8N -> Footprints:PSON65P250X250X100-8N
- U7: footprint MAX4466EXK:SOT65P210X110-5N -> Footprints:SOT65P210X110-5N
Other:
- note added: "(Q1)It has 3 pins in total we only connect 1 and 3."
- note added: "Envinormental sensor"
- note removed: "BME208"
- moved on the sheet: C15, C16, C17, C18, C19, C20, MK1, R17, R24, R25, R26, R27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

Commit message: finished_PCB
Changed lines of the file:
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@@
 		(on_board yes)
 		(dnp no)
-		(fields_autoplaced yes)
 		(property "Reference" "C23"
-			(at 209.55 59.6899 0)
+			(at 207.01 58.928 0)
 			(effects
 				(font
